File: SLiCAP/files/kicad/SLiCAP.kicad_sch (KiCad schematic)
At the start: 43 parts

Commit message: Version 4 update
Parts:
- removed A?: ~, symbol SLiCAP:Command
- F?, H? (x2): Vsource (none) -> ?
Other:
- note added: "C"
- note added: "Command"
- note added: "D"
- note added: "E"
- note added: "EZ"
- note added: "F"
- note added: "G"
- note added: "GND"
- note added: "H"
- note added: "HZ"
- note added: "I"
- note added: "J"
- note added: "J_noise"
- note added: "K"
- note added: "L"
- note added: "M"
- note added: "M-noise"
- note added: "N"
- note added: "N_dcvar"
- note added: "N_noise"
- note added: "O"
- note added: "O_dcvar"
- note added: "O_noise"
- note added: "Q"
- note added: "Q_noise"
- note added: "R"
- note added: "T"
- note added: "V"
- note added: "W"
- note added: "XJ"
- note added: "XM"
- note added: "XMD"
- note added: "XMPN"
- note added: "XMV"
- note added: "XQ"
- note added: "XQD"
- note added: "Xamp3"
- note added: "Xamp4"
- note added: "Xamp5"
- note added: "Xio3"
- note added: "Xio4"
- note added: "Xio5"
- note added: "r"
- moved on the sheet: A?, E?, G?, I?, J?, K?, L?, M?, N?, O1, Q?, R?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
Changed lines of the file:
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@@
 (kicad_sch
-	(version 20231120)
+	(version 20250114)
 	(generator "eeschema")
-	(generator_version "8.0")
+	(generator_version "9.0")
 	(paper "A4")
 	(title_block
